File: schematics/picalarm.kicad_pcb (KiCad board)
At the start: 2 copper layers, 44 parts, among them Q1 Q_NPN_BCE, Q2 Q_NPN_BCE, Q3 Q_NPN_BCE, Q4 Q_NPN_BCE, Q5 Q_NPN_BCE, SW1 Hour, SW2 Minute, SW3 Alarm Set, SW4 Alarm On, U1 7Segment, U2 7Segment, U3 7Segment, U4 PIC16F15344, U5 7Segment, X1 32.768 KHz

Commit message: Some rearranging of PCB components
Parts:
- moved R15 151.0 mm to (261.6, 85.1), turned to 90 degrees
- moved Q1 150.3 mm to (50.8, 77.5)
- moved Q2 110.6 mm to (91.4, 77.5)
- moved D3 86.1 mm to (123.2, 57.1)
- moved R17 83.9 mm to (233.8, 126.3)
- moved R8 83.9 mm to (233.8, 123.3)
- moved R18 83.9 mm to (246.4, 113.8)
- moved R19 83.9 mm to (224.0, 146.2)
- moved R20 83.9 mm to (246.4, 116.8)
- moved R22 83.9 mm to (246.4, 122.9)
- moved R6 83.9 mm to (246.4, 110.7)
- moved SW1 83.9 mm to (224.4, 149.2)
- moved SW2 83.9 mm to (235.9, 129.4)
- moved R21 83.9 mm to (246.4, 119.9)
- moved SW3 83.9 mm to (235.9, 136.9)
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Connections:
- Q1 pad 1: Net-(Q1-Pad1) -> GND
- Q1 pad 3: GND -> Net-(Q1-Pad3)
- Q2 pad 1: Net-(Q2-Pad1) -> GND
- Q2 pad 3: GND -> Net-(Q2-Pad3)
- Q3 pad 1: Net-(Q3-Pad1) -> GND
- Q3 pad 3: GND -> Net-(Q3-Pad3)
- Q4 pad 1: Net-(Q4-Pad1) -> GND
- Q4 pad 2: Net-(BZ1-Pad2) -> Net-(Q4-Pad2)
- Q4 pad 3: GND -> Net-(BZ1-Pad2)
- Q5 pad 1: Net-(Q5-Pad1) -> GND
- Q5 pad 3: GND -> Net-(Q5-Pad3)
- R11 pad 2: Net-(Q2-Pad1) -> Net-(Q2-Pad2)
- R14 pad 2: Net-(Q3-Pad1) -> Net-(Q3-Pad2)
- R15 pad 2: Net-(Q4-Pad1) -> Net-(Q4-Pad2)
- R16 pad 2: Net-(Q5-Pad1) -> Net-(Q5-Pad2)
- R2 pad 2: Net-(Q1-Pad1) -> Net-(Q1-Pad2)
- U1 pad 1: Net-(Q1-Pad2) -> Net-(Q1-Pad3)
- U1 pad 5: Net-(Q1-Pad2) -> Net-(Q1-Pad3)
- U2 pad 1: Net-(Q2-Pad2) -> Net-(Q2-Pad3)
- U2 pad 5: Net-(Q2-Pad2) -> Net-(Q2-Pad3)
- U3 pad 1: Net-(Q3-Pad2) -> Net-(Q3-Pad3)
- U3 pad 5: Net-(Q3-Pad2) -> Net-(Q3-Pad3)
- U5 pad 1: Net-(Q5-Pad2) -> Net-(Q5-Pad3)
- U5 pad 5: Net-(Q5-Pad2) -> Net-(Q5-Pad3)
- X1 pad 1: Net-(U4-Pad3) -> Net-(U4-Pad2)
- X1 pad 2: Net-(U4-Pad2) -> Net-(U4-Pad3)

Commit message: More rearranging of PCB components
Parts:
- added J1: USB_B_Mini, Connector_USB:USB_Micro-B_GCT_USB3076-30-A, B.Cu at (15.1, 61.1)
- C1, C2, D1, Q1, Q2, Q3, Q5, R1, R10, R11, R14, R16, R17, R18, R19, R2, R20, R21, R22, R23, R3, R4, R5, R6, R7, R8, R9, SW1, SW2, SW3, SW4, U4, X1: moved to B.Cu
- moved SW4 244.6 mm to (16.5, 12.7)
- moved SW1 243.1 mm to (15.2, 25.4)
- moved SW2 239.7 mm to (15.2, 35.6)
- moved SW3 238.7 mm to (15.2, 45.7)
- moved R17 154.9 mm to (109.2, 34.3)
- moved R20 150.1 mm to (119.4, 36.8)
- moved R21 134.8 mm to (142.2, 34.3)
- moved R22 133.5 mm to (142.2, 39.4)
- moved R19 130.5 mm to (142.2, 44.5)
- moved R18 120.5 mm to (153.7, 36.8)
- moved R23 108.1 mm to (153.7, 41.9)
- moved U4 81.8 mm to (138.4, 24.1), turned to 180 degrees
- moved C1 79.9 mm to (143.3, 20.8), turned to 270 degrees
- moved C2 79.9 mm to (147.1, 20.8), turned to 270 degrees
- moved X1 78.5 mm to (142.2, 26.7)
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Other:
- board outline added: 165.1 x 61 mm
