File: schematics/picalarm.sch (KiCad schematic (older format))
At the start: 7 parts, among them U1 PIC16F15344, U2 7Segment, U3 7Segment, U4 7Segment, U5 7Segment

Commit message: More schematics
Parts:
- added BZ1: Buzzer, symbol Device:Buzzer
- added C1, C2: idk uF, symbol Device:C_Small
- added D3: Red LED, symbol Device:LED
- added SW1: Hour, SW_1825910-6-4, symbol 1825910-6:1825910-6
- added SW2: Minute, SW_1825910-6-4, symbol 1825910-6:1825910-6
- added SW3: Alarm Set, SW_1825910-6-4, symbol 1825910-6:1825910-6
- added SW4: Alarm On, symbol Switch:SW_SPDT
- added X1: 32.768 KHz, symbol Device:Crystal
- D1, D2: value LED -> Red LED
Connections:
- net labels added: GNDREF
- wire segments 0 -> 13
Changed lines of the file:
@@
 EESchema Schematic File Version 4
+LIBS:picalarm-cache
 EELAYER 26 0
 EELAYER END
@@
 $EndComp
 $Comp
-L power:+5V #PWR?
+L power:+5V #PWR0101
 U 1 1 5BBF0ED6
 P 5050 1400
-F 0 "#PWR?" H 5050 1250 50  0001 C CNN
+F 0 "#PWR0101" H 5050 1250 50  0001 C CNN
 F 1 "+5V" H 5065 1573 50  0000 C CNN
 F 2 "" H 5050 1400 50  0001 C CNN
@@
 P 7000 2250
 F 0 "D1" V 7038 2133 50  0000 R CNN
-F 1 "LED" V 6947 2133 50  0000 R CNN
+F 1 "Red LED" V 6947 2133 50  0000 R CNN
 F 2 "" H 7000 2250 50  0001 C CNN
 F 3 "~" H 7000 2250 50  0001 C CNN
@@
 P 7000 2750
 F 0 "D2" V 7038 2633 50  0000 R CNN
-F 1 "LED" V 6947 2633 50  0000 R CNN
+F 1 "Red LED" V 6947 2633 50  0000 R CNN
 F 2 "" H 7000 2750 50  0001 C CNN
 F 3 "~" H 7000 2750 50  0001 C CNN
@@
 	0    -1   -1   0
 $EndComp
+$Comp
+L Device:Crystal X1
+U 1 1 5BBF9C25
+P 3100 3050
+F 0 "X1" V 3146 2919 50  0000 R CNN
+F 1 "32.768 KHz" V 3055 2919 50  0000 R CNN
+F 2 "" H 3100 3050 50  0001 C CNN
+F 3 "~" H 3100 3050 50  0001 C CNN
+	1    3100 3050
+	0    -1   -1   0
+$EndComp
+$Comp
+L Device:C_Small C2
+U 1 1 5BBF9D43
+P 2900 2800
+F 0 "C2" V 3129 2800 50  0000 C CNN
+F 1 "idk uF" V 3038 2800 50  0000 C CNN
+F 2 "" H 2900 2800 50  0001 C CNN
+F 3 "~" H 2900 2800 50  0001 C CNN
+	1    2900 2800
+	0    -1   -1   0
+$EndComp
+$Comp
+L Device:C_Small C1
+U 1 1 5BBF9D83
+P 2900 3300
+F 0 "C1" V 3129 3300 50  0000 C CNN
+F 1 "idk uF" V 3038 3300 50  0000 C CNN
+F 2 "" H 2900 3300 50  0001 C CNN
+F 3 "~" H 2900 3300 50  0001 C CNN
+	1    2900 3300
+	0    -1   -1   0
+$EndComp
+Wire Wire Line
+	3000 2800 3100 2800
+Wire Wire Line
+	3100 2800 3100 2900
+Connection ~ 3100 2800
+Wire Wire Line
+	3100 2800 3550 2800
+$Comp
+L power:GNDREF #PWR0102
+U 1 1 5BBFA1EA
+P 2500 3150
+F 0 "#PWR0102" H 2500 2900 50  0001 C CNN
+F 1 "GNDREF" H 2505 2977 50  0001 C CNN
+F 2 "" H 2500 3150 50  0001 C CNN
+F 3 "" H 2500 3150 50  0001 C CNN
+	1    2500 3150
+	1    0    0    -1
+$EndComp
+Wire Wire Line
+	2500 3150 2500 3050
+Wire Wire Line
+	2500 3050 2700 3050
+Connection ~ 2700 3050
+Wire Wire Line
+	2700 3050 2700 2800
+$Comp
+L Switch:SW_SPDT SW4
+U 1 1 5BBFA913
+P 1450 2850
+F 0 "SW4" H 1450 2525 50  0000 C CNN
+F 1 "Alarm On" H 1450 2616 50  0000 C CNN
+F 2 "" H 1450 2850 50  0001 C CNN
+F 3 "" H 1450 2850 50  0001 C CNN
+	1    1450 2850
+	-1   0    0    1
+$EndComp
+$Comp
+L power:GNDREF #PWR0103
+U 1 1 5BBFAC09
+P 4200 3350
+F 0 "#PWR0103" H 4200 3100 50  0001 C CNN
+F 1 "GNDREF" H 4205 3177 50  0001 C CNN
+F 2 "" H 4200 3350 50  0001 C CNN
+F 3 "" H 4200 3350 50  0001 C CNN
+	1    4200 3350
+	1    0    0    -1
+$EndComp
+Wire Wire Line
+	2700 3300 2700 3050
+Wire Wire Line
+	3550 2900 3550 3300
+Wire Wire Line
+	3000 3300 3100 3300
+Wire Wire Line
+	3100 3200 3100 3300
+Connection ~ 3100 3300
+Wire Wire Line
+	3100 3300 3550 3300
+Wire Wire Line
+	2700 3300 2800 3300
+Wire Wire Line
+	2800 2800 2700 2800
+$Comp
+L Device:LED D3
+U 1 1 5BBFC348
+P 1000 2950
+F 0 "D3" H 991 3166 50  0000 C CNN
+F 1 "Red LED" H 991 3075 50  0000 C CNN
+F 2 "" H 1000 2950 50  0001 C CNN
+F 3 "~" H 1000 2950 50  0001 C CNN
+	1    1000 2950
+	1    0    0    -1
+$EndComp
+$Comp
+L Device:Buzzer BZ1
+U 1 1 5BBFC3D9
+P 4700 3600
+F 0 "BZ1" H 4853 3629 50  0000 L CNN
+F 1 "Buzzer" H 4853 3538 50  0000 L CNN
+F 2 "" V 4675 3700 50  0001 C CNN
+F 3 "~" V 4675 3700 50  0001 C CNN
+	1    4700 3600
+	1    0    0    -1
+$EndComp
+$Comp
+L 1825910-6:1825910-6 SW1
+U 1 1 5BBFCCCB
+P 1450 1000
+F 0 "SW1" H 1450 1365 50  0000 C CNN
+F 1 "Hour" H 1450 1274 50  0000 C CNN
+F 2 "SW_1825910-6-4" H 1450 1000 50  0001 L BNN
+F 3 "1825910-6" H 1450 1000 50  0001 L BNN
+F 4 "FSM4JH=6MM TACT SWITCH, HIGH TEMP" H 1450 1000 50  0001 L BNN "Field4"
+F 5 "1825910-6" H 1450 1000 50  0001 L BNN "Field5"
+F 6 "http://www.te.com/usa-en/product-1825910-6.html" H 1450 1000 50  0001 L BNN "Field6"
+F 7 "Compliant" H 1450 1000 50  0001 L BNN "Field7"
+F 8 "50 mA" H 1450 1000 50  0001 L BNN "Field8"
+F 9 "450-1650-ND" H 1450 1000 50  0001 L BNN "Field9"
+F 10 "https://www.digikey.ca/product-detail/en/te-connectivity-alcoswitch-switches/1825910-6/450-1650-ND/1632536?utm_source=snapeda&utm_medium=aggregator&utm_campaign=symbol" H 1450 1000 50  0001 L BNN "Field10"
+F 11 "Single Pole - Single Throw" H 1450 1000 50  0001 L BNN "Field11"
+F 12 "TE Connectivity" H 1450 1000 50  0001 L BNN "Field12"
+F 13 "None" H 1450 1000 50  0001 L BNN "Field13"
+	1    1450 1000
+	1    0    0    -1
+$EndComp
+$Comp
+L 1825910-6:1825910-6 SW2
+U 1 1 5BBFCD93
+P 1450 1600
+F 0 "SW2" H 1450 1965 50  0000 C CNN
+F 1 "Minute" H 1450 1874 50  0000 C CNN
+F 2 "SW_1825910-6-4" H 1450 1600 50  0001 L BNN
+F 3 "1825910-6" H 1450 1600 50  0001 L BNN
+F 4 "FSM4JH=6MM TACT SWITCH, HIGH TEMP" H 1450 1600 50  0001 L BNN "Field4"
+F 5 "1825910-6" H 1450 1600 50  0001 L BNN "Field5"
+F 6 "http://www.te.com/usa-en/product-1825910-6.html" H 1450 1600 50  0001 L BNN "Field6"
+F 7 "Compliant" H 1450 1600 50  0001 L BNN "Field7"
+F 8 "50 mA" H 1450 1600 50  0001 L BNN "Field8"
+F 9 "450-1650-ND" H 1450 1600 50  0001 L BNN "Field9"
+F 10 "https://www.digikey.ca/product-detail/en/te-connectivity-alcoswitch-switches/1825910-6/450-1650-ND/1632536?utm_source=snapeda&utm_medium=aggregator&utm_campaign=symbol" H 1450 1600 50  0001 L BNN "Field10"
+F 11 "Single Pole - Single Throw" H 1450 1600 50  0001 L BNN "Field11"
+F 12 "TE Connectivity" H 1450 1600 50  0001 L BNN "Field12"
+F 13 "None" H 1450 1600 50  0001 L BNN "Field13"
+	1    1450 1600
+	1    0    0    -1
+$EndComp
+$Comp
+L 1825910-6:1825910-6 SW3
+U 1 1 5BBFCE47
+P 1450 2250
+F 0 "SW3" H 1450 2615 50  0000 C CNN
+F 1 "Alarm Set" H 1450 2524 50  0000 C CNN
+F 2 "SW_1825910-6-4" H 1450 2250 50  0001 L BNN
+F 3 "1825910-6" H 1450 2250 50  0001 L BNN
+F 4 "FSM4JH=6MM TACT SWITCH, HIGH TEMP" H 1450 2250 50  0001 L BNN "Field4"
+F 5 "1825910-6" H 1450 2250 50  0001 L BNN "Field5"
+F 6 "http://www.te.com/usa-en/product-1825910-6.html" H 1450 2250 50  0001 L BNN "Field6"
+F 7 "Compliant" H 1450 2250 50  0001 L BNN "Field7"
+F 8 "50 mA" H 1450 2250 50  0001 L BNN "Field8"
+F 9 "450-1650-ND" H 1450 2250 50  0001 L BNN "Field9"
+F 10 "https://www.digikey.ca/product-detail/en/te-connectivity-alcoswitch-switches/1825910-6/450-1650-ND/1632536?utm_source=snapeda&utm_medium=aggregator&utm_campaign=symbol" H 1450 2250 50  0001 L BNN "Field10"
+F 11 "Single Pole - Single Throw" H 1450 2250 50  0001 L BNN "Field11"
+F 12 "TE Connectivity" H 1450 2250 50  0001 L BNN "Field12"
+F 13 "None" H 1450 2250 50  0001 L BNN "Field13"
+	1    1450 2250
+	1    0    0    -1
+$EndComp
 $EndSCHEMATC

Commit message: Completed schematic
Parts:
- removed C1, C2: idk uF, symbol Device:C_Small
- removed SW1: Hour, SW_1825910-6-4, symbol 1825910-6:1825910-6
- removed SW2: Minute, SW_1825910-6-4, symbol 1825910-6:1825910-6
- removed SW3: Alarm Set, SW_1825910-6-4, symbol 1825910-6:1825910-6
- added C3: 0.1µF, symbol Device:C_Small
- added C4: 0.01µF, symbol Device:C_Small
- added Q1, Q2, Q3, Q4, Q5: Q_NPN_BCE, symbol Device:Q_NPN_BCE
- added R1, R2, R21, R23, R3, R4, R5, R6: 10k, symbol Device:R_US
- added R10, R11, R12, R9: 10K, symbol Device:R_US
- added R13, R14, R15, R16, R17, R18, R19: 100R, symbol Device:R_US
- added R20: 1K, symbol Device:R_US
- added R22, R7, R8: 160R, symbol Device:R_US
- added SW1: Hour, symbol Switch:SW_Push
- added SW2: Minute, symbol Switch:SW_Push
- added SW3: Alarm Set, symbol Switch:SW_Push
Connections:
- net labels added: BTN_ALARM_ADJUST, BTN_HOUR, BTN_MINUTE, CATH_HOURS_ONES, CATH_HOURS_TENS, CATH_MINUTES_ONES, CATH_MINUTES_TENS, GND, SEGMENT_A, SEGMENT_B, SEGMENT_C, SEGMENT_D, SEGMENT_E, SEGMENT_F, SEGMENT_G, SWT_ALARM, VDD
- net labels removed: +5V, GNDREF
- wire segments 13 -> 42

Commit message: Generated netlist and PCB stub
Parts:
- BZ1: footprint (none) -> Buzzer_Beeper:Buzzer_12x9.5RM7.6
- C1: renamed from C3; footprint (none) -> Capacitor_THT:C_Disc_D3.0mm_W1.6mm_P2.50mm
- C2: renamed from C4; footprint (none) -> Capacitor_THT:C_Disc_D3.0mm_W1.6mm_P2.50mm
- D1: renamed from D3; footprint (none) -> LED_THT:LED_D4.0mm
- D2: renamed from D1; footprint (none) -> LED_THT:LED_D4.0mm
- D3: renamed from D2; footprint (none) -> LED_THT:LED_D4.0mm
- Q1, Q2, Q3: footprint (none) -> Package_TO_SOT_THT:TO-92_Inline_Wide
- Q4: renamed from Q5; footprint (none) -> Package_TO_SOT_THT:TO-92_Inline_Wide
- Q5: renamed from Q4; footprint (none) -> Package_TO_SOT_THT:TO-92_Inline_Wide
- R1: renamed from R21; footprint (none) -> Resistor_THT:R_Axial_DIN0207_L6.3mm_D2.5mm_P7.62mm_Horizontal
- R10: renamed from R23; footprint (none) -> Resistor_THT:R_Axial_DIN0207_L6.3mm_D2.5mm_P7.62mm_Horizontal
- R11: renamed from R10; footprint (none) -> Resistor_THT:R_Axial_DIN0207_L6.3mm_D2.5mm_P7.62mm_Horizontal
- R12: renamed from R7; footprint (none) -> Resistor_THT:R_Axial_DIN0207_L6.3mm_D2.5mm_P7.62mm_Horizontal
- R13: renamed from R8; footprint (none) -> Resistor_THT:R_Axial_DIN0207_L6.3mm_D2.5mm_P7.62mm_Horizontal
- R14: renamed from R11; footprint (none) -> Resistor_THT:R_Axial_DIN0207_L6.3mm_D2.5mm_P7.62mm_Horizontal
- R15: renamed from R20; footprint (none) -> Resistor_THT:R_Axial_DIN0207_L6.3mm_D2.5mm_P7.62mm_Horizontal
- R16: renamed from R12; footprint (none) -> Resistor_THT:R_Axial_DIN0207_L6.3mm_D2.5mm_P7.62mm_Horizontal
- R17: renamed from R13; footprint (none) -> Resistor_THT:R_Axial_DIN0207_L6.3mm_D2.5mm_P7.62mm_Horizontal
- R18: renamed from R16; footprint (none) -> Resistor_THT:R_Axial_DIN0207_L6.3mm_D2.5mm_P7.62mm_Horizontal
- R19, R4: footprint (none) -> Resistor_THT:R_Axial_DIN0207_L6.3mm_D2.5mm_P7.62mm_Horizontal
- R2: renamed from R9; footprint (none) -> Resistor_THT:R_Axial_DIN0207_L6.3mm_D2.5mm_P7.62mm_Horizontal
- R20: renamed from R14; footprint (none) -> Resistor_THT:R_Axial_DIN0207_L6.3mm_D2.5mm_P7.62mm_Horizontal
- R21: renamed from R17; footprint (none) -> Resistor_THT:R_Axial_DIN0207_L6.3mm_D2.5mm_P7.62mm_Horizontal
- R22: renamed from R15; footprint (none) -> Resistor_THT:R_Axial_DIN0207_L6.3mm_D2.5mm_P7.62mm_Horizontal
- R23: renamed from R18; footprint (none) -> Resistor_THT:R_Axial_DIN0207_L6.3mm_D2.5mm_P7.62mm_Horizontal
- R3: renamed from R2; footprint (none) -> Resistor_THT:R_Axial_DIN0207_L6.3mm_D2.5mm_P7.62mm_Horizontal
- R5: renamed from R6; footprint (none) -> Resistor_THT:R_Axial_DIN0207_L6.3mm_D2.5mm_P7.62mm_Horizontal
- R6: renamed from R22; footprint (none) -> Resistor_THT:R_Axial_DIN0207_L6.3mm_D2.5mm_P7.62mm_Horizontal
- R7: renamed from R1; footprint (none) -> Resistor_THT:R_Axial_DIN0207_L6.3mm_D2.5mm_P7.62mm_Horizontal
- R8: renamed from R3; footprint (none) -> Resistor_THT:R_Axial_DIN0207_L6.3mm_D2.5mm_P7.62mm_Horizontal
- R9: renamed from R5; footprint (none) -> Resistor_THT:R_Axial_DIN0207_L6.3mm_D2.5mm_P7.62mm_Horizontal
- SW1, SW2, SW3: footprint (none) -> Button_Switch_THT:SW_PUSH_6mm
- SW4: footprint (none) -> Button_Switch_THT:SW_CuK_OS102011MA1QN1_SPDT_Angled
- U1: renamed from U2; footprint 7 segment display blue common cathode -> Display_7Segment:SBC18-11SURKCGKWA
- U2: renamed from U3; footprint 7 segment display blue common cathode -> Display_7Segment:SBC18-11SURKCGKWA
- U3: renamed from U4; footprint 7 segment display blue common cathode -> Display_7Segment:SBC18-11SURKCGKWA
- U4: renamed from U1; footprint (none) -> Package_DIP:DIP-20_W7.62mm
- U5: footprint 7 segment display blue common cathode -> Display_7Segment:SBC18-11SURKCGKWA
- X1: footprint (none) -> Crystal:Crystal_DS26_D2.0mm_L6.0mm_Horizontal

Commit message: Some rearranging of PCB components
Parts:
- Q1, Q2, Q3, Q4, Q5: symbol Device:Q_NPN_BCE -> Device:Q_NPN_EBC
Changed lines of the file:
@@
 F 3 "~" H 6250 2550 50  0001 C CNN
 	1    6250 2550
-	0    1    1    0
+	0    -1   -1   0
 $EndComp
 Wire Wire Line
@@
 Connection ~ 1900 1000
 $Comp
-L Device:Q_NPN_BCE Q1
+L Device:Q_NPN_EBC Q1
 U 1 1 5BC68F53
 P 2150 5950
@@
 $EndComp
 $Comp
-L Device:Q_NPN_BCE Q2
+L Device:Q_NPN_EBC Q2
 U 1 1 5BC68FB7
 P 3750 5950
@@
 $EndComp
 $Comp
-L Device:Q_NPN_BCE Q3
+L Device:Q_NPN_EBC Q3
 U 1 1 5BC69015
 P 6100 5950
@@
 $EndComp
 $Comp
-L Device:Q_NPN_BCE Q5
+L Device:Q_NPN_EBC Q5
 U 1 1 5BC6907D
 P 7850 5950
@@
 $EndComp
 $Comp
-L Device:Q_NPN_BCE Q4
+L Device:Q_NPN_EBC Q4
 U 1 1 5BCA4279
 P 7800 3450
 F 0 "Q4" H 7991 3496 50  0000 L CNN
-F 1 "Q_NPN_BCE" H 7991 3405 50  0000 L CNN
+F 1 "Q_NPN_BCE" H 7991 3405 50  0001 L CNN
 F 2 "Package_TO_SOT_THT:TO-92_Inline_Wide" H 8000 3550 50  0001 C CNN
 F 3 "~" H 7800 3450 50  0001 C CNN

Commit message: More rearranging of PCB components
Parts:
- added J1: USB_B_Mini, Connector_USB:USB_Micro-B_GCT_USB3076-30-A, symbol Connector:USB_B_Mini
Connections:
- wire segments 42 -> 44
- no-connect marks 0 -> 4
Changed lines of the file:
@@
 	1    0    0    -1
 $EndComp
+$Comp
+L Connector:USB_B_Mini J1
+U 1 1 5BCC48DE
+P 10050 1050
+F 0 "J1" H 10105 1517 50  0000 C CNN
+F 1 "USB_B_Mini" H 10105 1426 50  0000 C CNN
+F 2 "Connector_USB:USB_Micro-B_GCT_USB3076-30-A" H 10200 1000 50  0001 C CNN
+F 3 "~" H 10200 1000 50  0001 C CNN
+	1    10050 1050
+	1    0    0    -1
+$EndComp
+$Comp
+L power:VDD #PWR0101
+U 1 1 5BCC4983
+P 10450 750
+F 0 "#PWR0101" H 10450 600 50  0001 C CNN
+F 1 "VDD" H 10467 923 50  0000 C CNN
+F 2 "" H 10450 750 50  0001 C CNN
+F 3 "" H 10450 750 50  0001 C CNN
+	1    10450 750
+	1    0    0    -1
+$EndComp
+$Comp
+L power:GND #PWR0102
+U 1 1 5BCC4A14
+P 10050 1450
+F 0 "#PWR0102" H 10050 1200 50  0001 C CNN
+F 1 "GND" H 10055 1277 50  0001 C CNN
+F 2 "" H 10050 1450 50  0001 C CNN
+F 3 "" H 10050 1450 50  0001 C CNN
+	1    10050 1450
+	1    0    0    -1
+$EndComp
+Wire Wire Line
+	10350 850  10450 850
+Wire Wire Line
+	10450 850  10450 750
+NoConn ~ 10350 1050
+NoConn ~ 10350 1150
+NoConn ~ 10350 1250
+NoConn ~ 9950 1450
 $EndSCHEMATC
